File: pcb/raspberry_pi_hat/raspberry_pi_hat.sch (KiCad schematic (older format))
At the start: 32 parts, among them J1 I2C, J2 IMU, J3 Raspberry_Pi_2_3, J4 PWM, SW1 SW_Push, SW2 SW_Push, SW3 SW_Push

Commit message: Agrega modificaciones en el tamaño del PCB
Parts:
- R1, R10, R11, R12, R13, R14, R2, R3, R4, R5, R6, R7, R8, R9: footprint Resistor_THT:R_Axial_DIN0207_L6.3mm_D2.5mm_P10.16mm_Horizontal -> Resistor_THT:R_BIG_Axial_DIN0207
Changed lines of the file:
@@
 F 0 "R7" V 3725 3850 50  0000 L CNN
 F 1 "820" V 3650 3825 50  0000 L CNN
-F 2 "Resistor_THT:R_Axial_DIN0207_L6.3mm_D2.5mm_P10.16mm_Horizontal" V 3580 3900 50  0001 C CNN
+F 2 "Resistor_THT:R_BIG_Axial_DIN0207" V 3580 3900 50  0001 C CNN
 F 3 "~" H 3650 3900 50  0001 C CNN
 	1    3650 3900
@@
 F 0 "R8" V 3725 4075 50  0000 L CNN
 F 1 "820" V 3650 4050 50  0000 L CNN
-F 2 "Resistor_THT:R_Axial_DIN0207_L6.3mm_D2.5mm_P10.16mm_Horizontal" V 3580 4125 50  0001 C CNN
+F 2 "Resistor_THT:R_BIG_Axial_DIN0207" V 3580 4125 50  0001 C CNN
 F 3 "~" H 3650 4125 50  0001 C CNN
 	1    3650 4125
@@
 F 0 "R9" V 3725 4325 50  0000 L CNN
 F 1 "820" V 3650 4300 50  0000 L CNN
-F 2 "Resistor_THT:R_Axial_DIN0207_L6.3mm_D2.5mm_P10.16mm_Horizontal" V 3580 4375 50  0001 C CNN
+F 2 "Resistor_THT:R_BIG_Axial_DIN0207" V 3580 4375 50  0001 C CNN
 F 3 "~" H 3650 4375 50  0001 C CNN
 	1    3650 4375
@@
 F 0 "R10" V 3725 4550 50  0000 L CNN
 F 1 "820" V 3650 4525 50  0000 L CNN
-F 2 "Resistor_THT:R_Axial_DIN0207_L6.3mm_D2.5mm_P10.16mm_Horizontal" V 3580 4600 50  0001 C CNN
+F 2 "Resistor_THT:R_BIG_Axial_DIN0207" V 3580 4600 50  0001 C CNN
 F 3 "~" H 3650 4600 50  0001 C CNN
 	1    3650 4600
@@
 F 0 "R11" V 3725 4775 50  0000 L CNN
 F 1 "820" V 3650 4750 50  0000 L CNN
-F 2 "Resistor_THT:R_Axial_DIN0207_L6.3mm_D2.5mm_P10.16mm_Horizontal" V 3580 4825 50  0001 C CNN
+F 2 "Resistor_THT:R_BIG_Axial_DIN0207" V 3580 4825 50  0001 C CNN
 F 3 "~" H 3650 4825 50  0001 C CNN
 	1    3650 4825
@@
 F 0 "R12" V 3725 5000 50  0000 L CNN
 F 1 "820" V 3650 4975 50  0000 L CNN
-F 2 "Resistor_THT:R_Axial_DIN0207_L6.3mm_D2.5mm_P10.16mm_Horizontal" V 3580 5050 50  0001 C CNN
+F 2 "Resistor_THT:R_BIG_Axial_DIN0207" V 3580 5050 50  0001 C CNN
 F 3 "~" H 3650 5050 50  0001 C CNN
 	1    3650 5050
@@
 F 0 "R13" V 3725 5225 50  0000 L CNN
 F 1 "820" V 3650 5200 50  0000 L CNN
-F 2 "Resistor_THT:R_Axial_DIN0207_L6.3mm_D2.5mm_P10.16mm_Horizontal" V 3580 5275 50  0001 C CNN
+F 2 "Resistor_THT:R_BIG_Axial_DIN0207" V 3580 5275 50  0001 C CNN
 F 3 "~" H 3650 5275 50  0001 C CNN
 	1    3650 5275
@@
 F 0 "R14" V 3725 5450 50  0000 L CNN
 F 1 "820" V 3650 5425 50  0000 L CNN
-F 2 "Resistor_THT:R_Axial_DIN0207_L6.3mm_D2.5mm_P10.16mm_Horizontal" V 3580 5500 50  0001 C CNN
+F 2 "Resistor_THT:R_BIG_Axial_DIN0207" V 3580 5500 50  0001 C CNN
 F 3 "~" H 3650 5500 50  0001 C CNN
 	1    3650 5500
@@
 F 0 "R2" V 3050 2325 50  0000 L CNN
 F 1 "10k" V 2875 2300 50  0000 L CNN
-F 2 "Resistor_THT:R_Axial_DIN0207_L6.3mm_D2.5mm_P10.16mm_Horizontal" V 2905 2375 50  0001 C CNN
+F 2 "Resistor_THT:R_BIG_Axial_DIN0207" V 2905 2375 50  0001 C CNN
 F 3 "~" H 2975 2375 50  0001 C CNN
 	1    2975 2375
@@
 F 0 "R1" V 2725 2600 50  0000 L CNN
 F 1 "100k" V 2550 2550 50  0000 L CNN
-F 2 "Resistor_THT:R_Axial_DIN0207_L6.3mm_D2.5mm_P10.16mm_Horizontal" V 2580 2650 50  0001 C CNN
+F 2 "Resistor_THT:R_BIG_Axial_DIN0207" V 2580 2650 50  0001 C CNN
 F 3 "~" H 2650 2650 50  0001 C CNN
 	1    2650 2650
@@
 F 0 "R4" V 4175 2325 50  0000 L CNN
 F 1 "10k" V 4000 2300 50  0000 L CNN
-F 2 "Resistor_THT:R_Axial_DIN0207_L6.3mm_D2.5mm_P10.16mm_Horizontal" V 4030 2375 50  0001 C CNN
+F 2 "Resistor_THT:R_BIG_Axial_DIN0207" V 4030 2375 50  0001 C CNN
 F 3 "~" H 4100 2375 50  0001 C CNN
 	1    4100 2375
@@
 F 0 "R3" V 3850 2600 50  0000 L CNN
 F 1 "100k" V 3675 2550 50  0000 L CNN
-F 2 "Resistor_THT:R_Axial_DIN0207_L6.3mm_D2.5mm_P10.16mm_Horizontal" V 3705 2650 50  0001 C CNN
+F 2 "Resistor_THT:R_BIG_Axial_DIN0207" V 3705 2650 50  0001 C CNN
 F 3 "~" H 3775 2650 50  0001 C CNN
 	1    3775 2650
@@
 F 0 "R6" V 5225 2325 50  0000 L CNN
 F 1 "10k" V 5050 2300 50  0000 L CNN
-F 2 "Resistor_THT:R_Axial_DIN0207_L6.3mm_D2.5mm_P10.16mm_Horizontal" V 5080 2375 50  0001 C CNN
+F 2 "Resistor_THT:R_BIG_Axial_DIN0207" V 5080 2375 50  0001 C CNN
 F 3 "~" H 5150 2375 50  0001 C CNN
 	1    5150 2375
@@
 F 0 "R5" V 4900 2600 50  0000 L CNN
 F 1 "100k" V 4725 2550 50  0000 L CNN
-F 2 "Resistor_THT:R_Axial_DIN0207_L6.3mm_D2.5mm_P10.16mm_Horizontal" V 4755 2650 50  0001 C CNN
+F 2 "Resistor_THT:R_BIG_Axial_DIN0207" V 4755 2650 50  0001 C CNN
 F 3 "~" H 4825 2650 50  0001 C CNN
 	1    4825 2650
